Commit message: fixed incorrect urdf joint motion range

File: src/duco_support/urdf/duco_gcr5_910.urdf (robot description, URDF)
Before this commit: robot gcr5_910, 7 links, 6 joints
Joints:
- joint arm_1_joint_1: limit lower=-3.1415926 upper=3.1415926 effort=194 velocity=3.926990817 -> lower=-6.2831853 upper=6.2831853 effort=194 velocity=3.926990817
- joint arm_1_joint_2: limit lower=-3.1415926 upper=3.1415926 effort=194 velocity=3.926990817 -> lower=-6.2831853 upper=6.2831853 effort=194 velocity=3.926990817
- joint arm_1_joint_3: limit lower=-3.1415926 upper=3.1415926 effort=194 velocity=3.926990817 -> lower=-2.7925268 upper=2.7925268 effort=194 velocity=3.926990817
- joint arm_1_joint_4: limit lower=-3.1415926 upper=3.1415926 effort=34 velocity=3.926990817 -> lower=-6.2831853 upper=6.2831853 effort=34 velocity=3.926990817
- joint arm_1_joint_5: limit lower=-3.1415926 upper=3.1415926 effort=34 velocity=3.926990817 -> lower=-6.2831853 upper=6.2831853 effort=34 velocity=3.926990817
- joint arm_1_joint_6: limit lower=-3.1415926 upper=3.1415926 effort=34 velocity=3.926990817 -> lower=-6.2831853 upper=6.2831853 effort=34 velocity=3.926990817
